File: stm32f407-core.kicad_sch (KiCad schematic)
At the start: 20 parts, among them J1 Conn_01x18_MountingPin, J2 Conn_01x04, J3 Conn_02x25_Odd_Even, J4 Conn_02x25_Odd_Even, U1 STM32F407ZGTx

Commit message: add
Parts:
- added C14, C15: 10u/16V, symbol Device:C
- added R3: 10R, symbol Device:R
- C1: value 100n -> 100n/16V
- R1, R2: value 10k -> 10k/1%
Connections:
- net GND: now also C14.2, C15.2
- net VREF: now also R3.1
- new net VREF+: C14.1, C15.1, R3.2
Other:
- note added: "VREF+"
- moved on the sheet: R2
